File: hardware/console-pcb/console-a/console-a.kicad_sch (KiCad schematic)
At the start: 35 parts, among them J1 USB-C plug, J2 Screen 2.8in, SW1 PEC11R-4215F-S0024, SW2 Sign (A), SW3 Back (B), SW4 Device (X), SW5 Reject (Y), U1 Pico 2 W, U2 AP22653W6-7, U3 USBLC6-2SC6, U4 USBLC6-2SC6

Commit message: console-a: rotations that match JLCPCB's footprints
In JLCPCB's 3D preview the Pico 2 W lay across its pads, turned 90° and
off the board's edge: JLCPCB places each part by its own footprint, whose
zero rotation isn't always KiCad's. key-c's SOT-23-6 parts had the same
problem and were turned by hand in the preview, which no file records.

Every placed part's KiCad footprint was compared with JLCPCB's EasyEDA
one, matching pins by function (JLCPCB's LED calls its anode pin 1). The
turns needed go on the parts as "JLCPCB Rotation Offset" (JLC_ROT in
gen_console.py), and tools/keypcb adds that field to the rotation it
writes to cpl.csv:
- U1 Pico 2 W 180 -> 90, J1 plug 0 -> 270, U3/U4 USBLC6 0 -> 270,
  SW2-SW5 0 -> 270
- U2 AP22653 0 -> 180: uncorrected, IN, EN and OUT would land on the
  wrong pads

Parts without the field come out as before: key-c's and key-b's BOM and
CPL regenerate byte-identical. tools/keypcb check console-a: ERC 0, DRC
0, unconnected 0, parity clean.

Co-Authored-By: Claude Opus 5.5 <noreply@anthropic.com>
Claude-Session: https://claude.ai/code/session_01D7AK26Q7fPhkjbuWVid6KM
Parts:
- J1, SW2, SW3, SW4, SW5, U1, U3, U4: JLCPCB Rotation Offset (none) -> -90
- U2: JLCPCB Rotation Offset (none) -> 180
