File: hardware/console-a/console-a/console-a.kicad_sch (KiCad schematic)
At the start: 33 parts, among them J2 AFC07-S24FCA-00, J3 KEY PORT, Q1 SS8050, SW1 TS-1187A-B-A-B, SW2 TS-1187A-B-A-B, SW3 TS-1187A-B-A-B, SW4 TS-1187A-B-A-B, SW5 TS-1187A-B-A-B, SW6 TS-1187A-B-A-B, SW7 TS-1187A-B-A-B, SW8 TS-1187A-B-A-B, SW9 TS-1187A-B-A-B, U1 Pico 2 W, U2 TPS22945DCKR, U3 USBLC6-2SC6, U4 USBLC6-2SC6

Commit message: console-a: factory-soldered Pico option, and how to get the right panel
The same board and Gerbers, with a second assembly set in
fab/factory-pico/ where JLCPCB also solders U1, the Pico 2 W
(LCSC C42394205, Raspberry Pi SC1633), on the back. It needs two-sided
assembly and X-ray. The default fab/bom.csv and cpl.csv are unchanged.

- gen.py: U1's MPN is SC1633 (the Pico 2 W without headers; SC1634 has
  headers). An LCSC_FACTORY field carries the factory option, and U1 stays
  in the position file. Track geometry is identical (244 segments,
  77 vias), so the committed Gerber zip is kept.
- tools/keypcb fab: a board with LCSC_FACTORY parts also gets
  fab/factory-pico/{bom,cpl}.csv. The key boards are unaffected.
- README "Getting the right panel":
  - The identity of the right part.
  - Two sellers whose ZJY133T-IF05 datasheets match the pin table
    (Adafruit 4520, Smart Prototyping 102108 plug-in).
  - The look-alikes to reject, a per-batch check, and how panels get into
    each console (they can't go through JLCPCB).

Checked: ERC 0, DRC 0, 0 unconnected, parity clean, pin check passes. Not
checked: JLCPCB's bottom-side placement and price for the Pico (only their
quote shows it).

Co-Authored-By: Claude Opus 5.5 <noreply@anthropic.com>
Claude-Session: https://claude.ai/code/session_012wBec1er2qFD8SksgKkpb8
Parts:
- U1: LCSC_FACTORY (none) -> C42394205; MPN SC1634 -> SC1633
