File: hardware/console-usb/console-usb/console-usb.kicad_sch (KiCad schematic)
At the start: 55 parts, among them J1 USB-C, J2 LCD 1.14in FPC, J3 BENCH, Q1 AO3401A, Q2 SS8050, SW1 D0, SW2 D1, SW3 D2, SW4 RESET, U1 ESP32-S3FH4R2, U2 USBLC6-2SC6, U3 AMS1117-3.3, U4 CH340C, U5 ATECC608C-MAHDA-S, Y1 40MHz

Commit message: console-usb: every part placed, and 3D renders with the screen
The generator now also writes a 70 x 28 mm board with every part placed (not
routed), and with "render" has KiCad's 3D view draw it: top, three-quarter,
the back, and the panel lifted off. The panel is a body of our own (glass,
frame, foam pads, the ribbon folding under into J2) carrying the review page
from docs/quorum-ui/feather. KiCad's DRC checks the placement against
JLCPCB's limits, and the generator checks what sits under the glass.

J2 becomes console-s3's HDGC 0.5K-HX-8PWB ZIF: the FH12, about 2 mm tall,
didn't fit under the glass on its 2 mm tape. The S3 takes the plain QFN-56
footprint; the thermal-via one drills 0.2 mm, under JLCPCB's limit. The
TS-1187A and the HRO USB-C have no 3D models in KiCad 9.0.9, so the board
names a TL3342 and a GCT USB4105 for the pictures. README.md shows the
renders and says what in them isn't the real part.

Co-Authored-By: Claude Opus 5.5 <noreply@anthropic.com>
Claude-Session: https://claude.ai/code/session_01X3JYWQkjPoxm8rL4Nn6uyS
Parts:
- removed J2: LCD 1.14in FPC, Connector_FFC-FPC:Hirose_FH12-8S-0.5SH_1x08-1MP_P0.50mm_Horizontal, symbol Connector_Generic_MountingPin:Conn_01x08_MountingPin
- added J2: LCD 1.14in FPC, pqusb:FPC_ZIF_8P_P0.5mm_HDGC_0.5K-HX-8PWB, symbol Connector_Generic:Conn_01x08
- U1: footprint Package_DFN_QFN:QFN-56-1EP_7x7mm_P0.4mm_EP4x4mm_ThermalVias -> Package_DFN_QFN:QFN-56-1EP_7x7mm_P0.4mm_EP4x4mm
Connections:
- net +3V3: now also J2.7 (Pin_7)
- net GND: now also J2.2 (Pin_2)
- net LCD_CS: now also J2.8 (Pin_8)
- net LCD_DC: now also J2.4 (Pin_4)
- net LCD_LEDA: now also J2.1 (Pin_1)
- net LCD_MOSI: now also J2.5 (Pin_5)
- net LCD_RST: now also J2.3 (Pin_3)
- net LCD_SCK: now also J2.6 (Pin_6)
