File: hardware/feather-wing/wing-a/wing-a.kicad_sch (KiCad schematic)
At the start: 24 parts, among them J1 USB-C plug, J2 Feather 16-pin, J3 Feather 12-pin, U2 AP22653W6-7, U3 USBLC6-2SC6, U4 USBLC6-2SC6

Commit message: wing-a and wing-b: KiCad-clean, key-c P3's LED line, wing-b on a straddle plug
KiCad 10.0.6 found what the self-check couldn't: gen_wing.py's rotate(),
shared with console-pocket, turned parts clockwise on the page where
KiCad turns them counter-clockwise, so every part at 90 or 270 had its
pads swapped against its tracks. rotate() is KiCad's now and ROT's 90s
and 270s are swapped; round pads join only inside their circle; loose
via and track ends are dropped. console-pocket's README now says not to
order it until it is regenerated the same way.

Both wings carry key-c P3's LED: A8 and B8 joined as KEY_LED, driven
from D13 (the status LED pin) through R13, D3 for ESD; R14 to A0 not
fitted. No firmware change.

wing-b is redrawn around a SHOU HAN 24P straddle-mount plug (C3151751)
on a tab out of the 12-pin side, in place of GCT's USB4155.

tools/keypcb fill then check, both wings: ERC 0, DRC 0, 0 unconnected,
parity clean. Fab files and renders in each wing's fab/. Not ordered.

Co-Authored-By: Claude Opus 5.5 <noreply@anthropic.com>
Claude-Session: https://claude.ai/code/session_014mGuGD4x9Si2dmdRKbhRec
Parts:
- added D3: ESD5Z5V0, pqwing:D_SOD-523, symbol pqwing:D_TVS
- added R13, R14: 100, pqwing:R_0402, symbol pqwing:R
Connections:
- net GND: now also D3.2 (A)
- net LED_ALT: now reaches J2.5 (A0)
- net LED_ALT: now also R14.2
- net KEY_LED: now reaches J1.A8 (SBU1)
- net KEY_LED: now also J1.B8 (SBU2), D3.1 (K), R13.1, R14.1
- net LED_D13: now reaches J3.4 (D13)
- net LED_D13: now also R13.2
- no-connect marks 22 -> 18
Other:
- note added: "Bus links: R9/R10 fitted put the key on the Feather's SDA/SCL, the bus today's console image reads. R11/R12 instead give it a bus of its own on D11/D12, for a later image. Never fit both pairs. The key's LED (key-c P3, on SBU): R13 to D13, the console's status LED, or R14 to A0 for a later image. Never fit both."
- note removed: "Bus links: R9/R10 fitted put the key on the Feather's SDA/SCL, the bus today's console image reads. R11/R12 instead give it a bus of its own on D11/D12, for a later image. Never fit both pairs."
