File: hardware/feather-wing/wing-b/wing-b.kicad_sch (KiCad schematic)
At the start: 22 parts, among them J1 USB-C plug, right angle, J2 Feather 16-pin, J3 Feather 12-pin, U2 AP22653W6-7, U3 USBLC6-2SC6, U4 USBLC6-2SC6

Commit message: wing-a and wing-b: KiCad-clean, key-c P3's LED line, wing-b on a straddle plug
KiCad 10.0.6 found what the self-check couldn't: gen_wing.py's rotate(),
shared with console-pocket, turned parts clockwise on the page where
KiCad turns them counter-clockwise, so every part at 90 or 270 had its
pads swapped against its tracks. rotate() is KiCad's now and ROT's 90s
and 270s are swapped; round pads join only inside their circle; loose
via and track ends are dropped. console-pocket's README now says not to
order it until it is regenerated the same way.

Both wings carry key-c P3's LED: A8 and B8 joined as KEY_LED, driven
from D13 (the status LED pin) through R13, D3 for ESD; R14 to A0 not
fitted. No firmware change.

wing-b is redrawn around a SHOU HAN 24P straddle-mount plug (C3151751)
on a tab out of the 12-pin side, in place of GCT's USB4155.

tools/keypcb fill then check, both wings: ERC 0, DRC 0, 0 unconnected,
parity clean. Fab files and renders in each wing's fab/. Not ordered.

Co-Authored-By: Claude Opus 5.5 <noreply@anthropic.com>
Claude-Session: https://claude.ai/code/session_014mGuGD4x9Si2dmdRKbhRec
Parts:
- removed J1: USB-C plug, right angle, pqwing:USB_C_Plug_GCT_USB4155_Horizontal, symbol pqwing:USB_C_Plug_24P_RA
- added D3: ESD5Z5V0, pqwing:D_SOD-523, symbol pqwing:D_TVS
- added J1: USB-C plug, straddle mount, pqwing:USB_C_Plug_ShouHan_24P-GTJB_Straddle, symbol pqwing:USB_C_Plug_Straddle
- added R13, R14: 100, pqwing:R_0402, symbol pqwing:R
Connections:
- net CC1: now also J1.A5 (CC)
- net GND: now also D3.2 (A), J1.A1 (GND), J1.A12 (GND), J1.B1 (GND), J1.B12 (GND), J1.SH (SHIELD)
- net KEY_SCL: now also J1.A7 (D-)
- net KEY_SDA: now also J1.A6 (D+)
- net VKEY: now also J1.A4 (VBUS), J1.A9 (VBUS), J1.B4 (VBUS), J1.B9 (VBUS)
- net LED_D13: now reaches J3.4 (D13)
- net LED_D13: now also R13.2
- net LED_ALT: now reaches J2.5 (A0)
- net LED_ALT: now also R14.2
- new net KEY_LED: D3.1 (K), J1.A8 (SBU1), J1.B8 (SBU2), R13.1, R14.1
- no-connect marks 38 -> 30
Other:
- note added: "Bus links: R9/R10 fitted put the key on the Feather's SDA/SCL, the bus today's console image reads. R11/R12 instead give it a bus of its own on D11/D12, for a later image. Never fit both pairs. The key's LED (key-c P3, on SBU): R13 to D13, the console's status LED, or R14 to A0 for a later image. Never fit both."
- note added: "The Feather's two header rows, Adafruit's order from the USB end. 3V3 and GND power the wing; D5, D6, D9, D10 are new pins for the key port; SDA/SCL (GPIO3/4) or D11/D12 carry the key's bus, chosen by R9-R12."
- note added: "The console end of key-c, as console-a has it: - VKEY comes through U2: 80 mA limit, reverse blocking, discharged when off. Never straight from a GPIO. EN pulled up: on by default. - CC1 and CC2 read on their own ADC1 pins (D5, D6). Plugged straight in, a key shows 5.1k on both. - 2.2k pull-ups to VKEY, so a key that's off isn't powered through SDA/SCL. - U3/U4 rails on 3V3: the CC pull-ups can't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"
- note added: "key-c's USB-C socket carries I2C, not USB (hardware/key-pcb/PROPOSALS.md): SDA on D+ (A6), SCL on D- (A7), power on VBUS, a 5.1k Rd on each CC. This plug has no B6/B7; key-c joins A6/B6 and A7/B7 itself. Its VCONN (B5) meets the key's second Rd, so it reads as CC2."
- note removed: "Bus links: R9/R10 fitted put the key on the Feather's SDA/SCL, the bus today's console image reads. R11/R12 instead give it a bus of its own on D11/D12, for a later image. Never fit both pairs."
- note removed: "The Feather's two header rows, Adafruit's order from the USB end. 3V3 and GND power the wing; D5, D9, D10 are new pins for the key port; SDA/SCL (GPIO3/4) or D11/D12 carry the key's bus, chosen by R9-R12."
- note removed: "The console end of key-c, as console-a has it: - VKEY comes through U2: 80 mA limit, reverse blocking, discharged when off. Never straight from a GPIO. EN pulled up: on by default. - CC1 read on an ADC1 pin (D5). Plugged straight in, a key shows 5.1k on it whichever way up. U4's second pair is spare. - 2.2k pull-ups to VKEY, so a key that's off isn't powered through SDA/SCL. - U3/U4 rails on 3V3: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"
- note removed: "key-c's USB-C socket carries I2C, not USB (hardware/key-pcb/PROPOSALS.md): SDA on D+ (A6), SCL on D- (A7), power on VBUS, a 5.1k Rd on each CC. Only this plug's A row can be routed, and it is all a key needs: key-c joins its two rows. The B row is soldered for strength only."
