File: hardware/key-pcb/key-c-usbc/key-c-usbc.kicad_pcb (KiCad board)
At the start: 2 copper layers, 16 x 36 mm, 13 parts, among them J1 HC-TYPE-C-16P-01A, U1 ATECC608C-SSHDA, U2 USBLC6-2SC6

Commit message: key-c P3: a green LED on SBU2 that the console lights
P2 plus two parts: D1, a green 0603 LED (C72043) beside U2, and R3,
470 ohm (C25117), from the receptacle's B8 (SBU2) to D1's anode. R3 is
first from the pad, so it limits whatever a plug puts on SBU. Only B8 is
wired: A8 sits under SDA's via. The wings join their plug's A8 and B8 and
drive them from D13, the status LED pin, so the key's LED follows it with
no firmware change. A cable to a laptop carries no SBU: it stays dark.

gen_cd.py writes P3 (and was first checked to rebuild P2 exactly);
`tools/keypcb gen-cd key-c-usbc` now writes only that board. P2's files
as ordered move to fab/P2/. KiCad 10.0.6, tools/keypcb check key-c-usbc:
ERC 0, DRC 0, 0 unconnected, parity clean. Not ordered.

Co-Authored-By: Claude Opus 5.5 <noreply@anthropic.com>
Claude-Session: https://claude.ai/code/session_014mGuGD4x9Si2dmdRKbhRec
Parts:
- added D1: green, LED_SMD:LED_0603_1608Metric, F.Cu at (103.0, 122.4)
- added R3: 470, Resistor_SMD:R_0402_1005Metric, F.Cu at (103.0, 125.0)
- moved R1 0.46 mm to (105.1, 125.6), turned to 180 degrees
Connections:
- J1 pad B8: unconnected-(J1-SBU2-PadB8) -> /LED
Routing:
- net /LED: track 0.00 -> 6.09 mm
- net Net-(D1-A): track 0.00 -> 1.30 mm
- net GND: track 3.46 -> 4.38 mm, vias 14 -> 15
- net /CC1: track 2.95 -> 3.85 mm
Other:
- board text added: "key-c P3 2026-10"
- board text removed: "key-c P2 2026-10"
