File: hardware/key-pcb/key-c-usbc/key-c-usbc.kicad_sch (KiCad schematic)
At the start: 11 parts, among them J1 HC-TYPE-C-16P-01A, U1 ATECC608C-SSHDA, U2 USBLC6-2SC6

Commit message: key-c P3: a green LED on SBU2 that the console lights
P2 plus two parts: D1, a green 0603 LED (C72043) beside U2, and R3,
470 ohm (C25117), from the receptacle's B8 (SBU2) to D1's anode. R3 is
first from the pad, so it limits whatever a plug puts on SBU. Only B8 is
wired: A8 sits under SDA's via. The wings join their plug's A8 and B8 and
drive them from D13, the status LED pin, so the key's LED follows it with
no firmware change. A cable to a laptop carries no SBU: it stays dark.

gen_cd.py writes P3 (and was first checked to rebuild P2 exactly);
`tools/keypcb gen-cd key-c-usbc` now writes only that board. P2's files
as ordered move to fab/P2/. KiCad 10.0.6, tools/keypcb check key-c-usbc:
ERC 0, DRC 0, 0 unconnected, parity clean. Not ordered.

Co-Authored-By: Claude Opus 5.5 <noreply@anthropic.com>
Claude-Session: https://claude.ai/code/session_014mGuGD4x9Si2dmdRKbhRec
Parts:
- added D1: green, LED_SMD:LED_0603_1608Metric, symbol Device:LED
- added R3: 470, Resistor_SMD:R_0402_1005Metric, symbol Device:R
Connections:
- net GND: now also D1.1 (K)
- net LED: now reaches J1.B8 (SBU2)
- net LED: now also R3.1
- new net: D1.2 (A), R3.2
- no-connect marks 2 -> 1
Other:
- note added: "USB-C used as plain wires, no USB: VBUS = key VCC (console GP6, switched) D+ = SDA (GP4), D- = SCL (GP5) A6/B6 and A7/B7 are joined on the board, so a cable works either way up. CC1/CC2: 5.1k each to GND (USB-C's Rd). The console's GP7 pull-up on CC reads low when a key is attached: that is DETECT. SBU2 lights the LED (the console drives it); SBU1 is open."
- note removed: "USB-C used as plain wires, no USB: VBUS = key VCC (console GP6, switched) D+ = SDA (GP4), D- = SCL (GP5) A6/B6 and A7/B7 are joined on the board, so a cable works either way up. CC1/CC2: 5.1k each to GND (USB-C's Rd). The console's GP7 pull-up on CC reads low when a key is attached: that is DETECT. SBU1/SBU2 unused."
