File: hardware/console-s3/console-s3/console-s3.kicad_pcb (KiCad board)
At the start: 2 copper layers, 64 x 22.9 mm, 45 parts, among them J1 USB-C, J2 PANEL, Q1 S8050, Q2 AO3401A, SW1 D0, SW2 D1, SW3 D2, SW4 BOOT, SW5 RESET, U1 ESP32-S3-WROOM-1-N4R2, U2 ATECC608C, U3 ME6211C33, U4 USBLC6-2SC6

Commit message: console-s3: the ESP32-S3-WROOM-1-N8R2, as PicoQuorumKey
Both boards now name one module, C2913204: the same footprint, pins and
2 MB quad PSRAM as the N4R2, cheaper, and ten times the stock on
2026-10-24. The generator's constants and the routed KiCad files carry
the new part number and flash size; only hidden properties and the
schematic's note change. The module isn't in the Gerbers, BOM or CPL,
so the fab files stay as they are.

Co-Authored-By: Claude Opus 5.5 <noreply@anthropic.com>
Claude-Session: https://claude.ai/code/session_01XwHg4ToGz3n53Vasj6GisW
Parts:
- U1: value ESP32-S3-WROOM-1-N4R2 -> ESP32-S3-WROOM-1-N8R2
Changed lines of the file:
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@@
 			)
 		)
-		(property "Value" "ESP32-S3-WROOM-1-N4R2"
+		(property "Value" "ESP32-S3-WROOM-1-N8R2"
 			(at 0 -13.7 0)
 			(layer "B.Fab")
@@
 			)
 		)
-		(property "Description" "ESP32-S3 module, 4 MB flash, 2 MB quad PSRAM, on the back; JLCPCB C2913203 is Standard-only: hand-soldered"
+		(property "Description" "ESP32-S3 module, 8 MB flash, 2 MB quad PSRAM, on the back; JLCPCB C2913204 is Standard-only: hand-soldered"
 			(at 0 0 0)
 			(layer "B.Fab")
@@
 			)
 		)
-		(property "MPN" "ESP32-S3-WROOM-1-N4R2"
+		(property "MPN" "ESP32-S3-WROOM-1-N8R2"
 			(at 0 0 0)
 			(layer "B.Fab")
