File: hardware/console-s3/console-s3/console-s3.kicad_sch (KiCad schematic)
At the start: 43 parts, among them J1 USB-C, J2 PANEL, Q1 S8050, Q2 AO3401A, SW1 D0, SW2 D1, SW3 D2, SW4 BOOT, SW5 RESET, U1 ESP32-S3-WROOM-1-N4R2, U2 ATECC608C, U3 ME6211C33, U4 USBLC6-2SC6

Commit message: console-s3: the ESP32-S3-WROOM-1-N8R2, as PicoQuorumKey
Both boards now name one module, C2913204: the same footprint, pins and
2 MB quad PSRAM as the N4R2, cheaper, and ten times the stock on
2026-10-24. The generator's constants and the routed KiCad files carry
the new part number and flash size; only hidden properties and the
schematic's note change. The module isn't in the Gerbers, BOM or CPL,
so the fab files stay as they are.

Co-Authored-By: Claude Opus 5.5 <noreply@anthropic.com>
Claude-Session: https://claude.ai/code/session_01XwHg4ToGz3n53Vasj6GisW
Parts:
- U1: value ESP32-S3-WROOM-1-N4R2 -> ESP32-S3-WROOM-1-N8R2; MPN ESP32-S3-WROOM-1-N4R2 -> ESP32-S3-WROOM-1-N8R2
Other:
- note added: "ESP32-S3-WROOM-1-N8R2 on the back, hand-soldered. The Feather ESP32-S3 Reverse TFT's GPIOs (firmware/board.py, "feather-s3"), so today's console image runs unchanged. Never an R8 module: octal PSRAM takes GPIO35-37."
- note removed: "ESP32-S3-WROOM-1-N4R2 on the back, hand-soldered. The Feather ESP32-S3 Reverse TFT's GPIOs (firmware/board.py, "feather-s3"), so today's console image runs unchanged. Never an R8 module: octal PSRAM takes GPIO35-37."
Changed lines of the file:
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@@
 (symbol (lib_id "pqs3:ESP32-S3-WROOM-1") (at 147.32 85.09 0) (unit 1) (exclude_from_sim no) (in_bom no) (on_board yes) (dnp no)
 (property "Reference" "U1" (at 151.13 55.88 0) (effects (font (size 1.27 1.27)) (justify left)))
-(property "Value" "ESP32-S3-WROOM-1-N4R2" (at 151.13 115.57000000000001 0) (effects (font (size 1.27 1.27)) (justify left)))
+(property "Value" "ESP32-S3-WROOM-1-N8R2" (at 151.13 115.57000000000001 0) (effects (font (size 1.27 1.27)) (justify left)))
 (property "Footprint" "pqs3:ESP32-S3-WROOM-1" (at 147.32 85.09 0) (effects (font (size 1.27 1.27)) (hide yes)))
 (property "Datasheet" "https://www.espressif.com/sites/default/files/documentation/esp32-s3-wroom-1_wroom-1u_datasheet_en.pdf" (at 147.32 85.09 0) (effects (font (size 1.27 1.27)) (hide yes)))
-(property "MPN" "ESP32-S3-WROOM-1-N4R2" (at 147.32 85.09 0) (effects (font (size 1.27 1.27)) (hide yes)))
-(property "Description" "ESP32-S3 module, 4 MB flash, 2 MB quad PSRAM, on the back; JLCPCB C2913203 is Standard-only: hand-soldered" (at 147.32 85.09 0) (effects (font (size 1.27 1.27)) (hide yes)))
+(property "MPN" "ESP32-S3-WROOM-1-N8R2" (at 147.32 85.09 0) (effects (font (size 1.27 1.27)) (hide yes)))
+(property "Description" "ESP32-S3 module, 8 MB flash, 2 MB quad PSRAM, on the back; JLCPCB C2913204 is Standard-only: hand-soldered" (at 147.32 85.09 0) (effects (font (size 1.27 1.27)) (hide yes)))
 (pin "1") (pin "2") (pin "3") (pin "4") (pin "5") (pin "6") (pin "7") (pin "8") (pin "9") (pin "10") (pin "11") (pin "12") (pin "13") (pin "14") (pin "15") (pin "16") (pin "17") (pin "18") (pin "19") (pin "20") (pin "21") (pin "22") (pin "23") (pin "24") (pin "25") (pin "26") (pin "27") (pin "28") (pin "29") (pin "30") (pin "31") (pin "32") (pin "33") (pin "34") (pin "35") (pin "36") (pin "37") (pin "38") (pin "39") (pin "40") (pin "41")
 (instances (project "console-s3" (path "/6216c6e8-43cf-4e09-8f97-aa6ffc48f7cc" (reference "U1") (unit 1)))))
@@
 (pin "1")
 (instances (project "console-s3" (path "/6216c6e8-43cf-4e09-8f97-aa6ffc48f7cc" (reference "#PWR004") (unit 1)))))
-(text "ESP32-S3-WROOM-1-N4R2 on the back, hand-soldered.\nThe Feather ESP32-S3 Reverse TFT's GPIOs (firmware/board.py,\n\"feather-s3\"), so today's console image runs unchanged.\nNever an R8 module: octal PSRAM takes GPIO35-37." (exclude_from_sim no) (at 127.0 123.19 0) (effects (font (size 1.27 1.27)) (justify left top)))
+(text "ESP32-S3-WROOM-1-N8R2 on the back, hand-soldered.\nThe Feather ESP32-S3 Reverse TFT's GPIOs (firmware/board.py,\n\"feather-s3\"), so today's console image runs unchanged.\nNever an R8 module: octal PSRAM takes GPIO35-37." (exclude_from_sim no) (at 127.0 123.19 0) (effects (font (size 1.27 1.27)) (justify left top)))
 (symbol (lib_id "pqs3:GND") (at 22.86 20.32 0) (unit 1) (exclude_from_sim no) (in_bom yes) (on_board yes) (dnp no)
 (property "Reference" "#PWR005" (at 22.86 20.32 0) (effects (font (size 1.27 1.27)) (hide yes)))
