File: hardware/console-s3/console-s3/console-s3.kicad_sch (KiCad schematic)
At the start: 43 parts, among them J1 USB-C, J2 PANEL, Q1 S8050, Q2 AO3401A, SW1 D0, SW2 D1, SW3 D2, SW4 PREV, SW5 BACK, U1 ESP32-S3-WROOM-1-N4R2, U2 ATECC608C, U3 ME6211C33, U4 USBLC6-2SC6

Commit message: console-s3: routed with Freerouting, brand silkscreen, BOOT and RESET
tools/keypcb route console-s3 routes the placed board with Freerouting
2.5 through KiCad's Specctra files, then drops dangling vias, stitches
ground and fills. The generator writes the board placed, plus locked
escape tracks for J1's USB pads and U2's bus. 537 tracks, 1066 mm, 70
vias (19 stitching).

- C5 turned toward U2; U4 moved; USB split at U4 (USB_DP/DN on J1's
  side, S3_DP/DN on the module's); 2.5 mm no-track rings round H1/H2.
- The silkscreen: the name traced from Atkinson Hyperlegible Next Bold
  (wordmark.py), the logos, and under the glass an 8-bit key below U2
  with a dragon guarding it, after Adventure (Atari 2600).
- The two right-hand buttons are BOOT (GPIO0, beside D0) and RESET (EN
  to ground) in place of PREV and BACK. The image never read those.
- Text 1.0 mm with 0.15 strokes; the project rules raised to match.

console-pocket's rotate(), which this generator shares, is fixed as on
claude/wing-a-refine (the same change on both branches).

KiCad 10.0.6, tools/keypcb check console-s3: ERC 0/0, DRC 0, 0
unconnected, 0 parity issues. Fab files in console-s3/fab/. Not ordered.
No firmware change.

Co-Authored-By: Claude Opus 5.5 <noreply@anthropic.com>
Claude-Session: https://claude.ai/code/session_014mGuGD4x9Si2dmdRKbhRec
Parts:
- SW4: value PREV -> BOOT
- SW5: value BACK -> RESET
Connections:
- net BTN_D0: now also SW4.1
- net EN: now also SW5.1
- net USB_DN: no longer U1.13 (IO19), U4.3 (IO2)
- net USB_DP: no longer U1.14 (IO20), U4.1 (IO1)
- net BTN_BACK: no longer names the net of U1.6 (IO6)
- net BTN_BACK: no longer SW5.1
- net BTN_PREV: no longer names the net of U1.5 (IO5)
- net BTN_PREV: no longer SW4.1
- new net S3_DN: U1.13 (IO19), U4.3 (IO2)
- new net S3_DP: U1.14 (IO20), U4.1 (IO1)
- no-connect marks 25 -> 27
Other:
- note added: "D0, D1, D2: the Feather's buttons on its GPIOs. D0 is BOOT: low when pressed, R5 up. D1, D2 high when pressed, R6 and R7 down. BOOT is D0 again; RESET pulls EN low."
- note added: "ESP32-S3-WROOM-1-N4R2 on the back, hand-soldered. The Feather ESP32-S3 Reverse TFT's GPIOs (firmware/board.py, "feather-s3"), so today's console image runs unchanged. Never an R8 module: octal PSRAM takes GPIO35-37."
- note removed: "D0, D1, D2: the Feather's buttons on its GPIOs. D0 is BOOT: low when pressed, R5 up. D1, D2 high when pressed, R6 and R7 down. PREV and BACK pull low on the S3's internal pull-ups."
- note removed: "ESP32-S3-WROOM-1-N4R2 on the back, hand-soldered. The Feather ESP32-S3 Reverse TFT's GPIOs (firmware/board.py, "feather-s3"), so today's console image runs unchanged. PREV (GPIO5) and BACK (GPIO6) are new: no image reads them yet. Never an R8 module: octal PSRAM takes GPIO35-37."

Commit message: console-s3: backlight from VBUS, longer module pads, J2 at the 21 mm reach
- The backlight was likely over-driven: 10 R from 3.3 V gave 20-40 mA against the
  panel's 20 mA maximum (ER-TFT1.14-2). It now runs from VBUS through 150 R
  (C22808): (5 - 3.0) V / 150 R = 13 mA, 16 mA at worst. Q2 and R4 move to VBUS.
- The module's pads reached 0.45 mm past its edge; they now reach 1.45 mm, as on
  PicoQuorumKey, for the iron. The courtyard and pin-1 dot follow.
- J2 moves to x 30.0, for the datasheet's folded reach of 21.0 +/- 0.5 mm from the
  glass's edge (it was 4.7 mm shorter). C6, the key and dragon art move with it, and
  the 3D fit models the fold from the same drawing.
- Placed, routed and checked again: ERC 0, DRC 0, parity 0; tools/keypcb jlc
  passes, its self-test 10/10; golden images rewritten.
- DESIGN.md drops the stale "No reset button" note: BOOT and RESET are on the board.

Co-Authored-By: Claude Opus 5.5 <noreply@anthropic.com>
Claude-Session: https://claude.ai/code/session_014mGuGD4x9Si2dmdRKbhRec
Parts:
- R1: value 10R -> 150R; LCSC C22859 -> C22808
Connections:
- net +3V3: no longer Q2.2 (S), R4.1
- net VBUS: now also Q2.2 (S), R4.1
Other:
- note added: "The panel: 1.14in 240x135 ST7789 on an 8-pin 0.5 mm ribbon, one seller's pin order (DESIGN.md). Its LEDK is GND inside, so Q2 switches LEDA from VBUS on the high side, R1 setting 13 mA; GPIO45 high is on, as on the Feather. R3 holds GPIO45 (a strap: VDD_SPI) low at reset."
- note removed: "The panel: 1.14in 240x135 ST7789 on an 8-pin 0.5 mm ribbon, one seller's pin order (DESIGN.md). Its LEDK is GND inside, so Q2 switches LEDA on the high side; GPIO45 high is on, as on the Feather. R3 holds GPIO45 (a strap: VDD_SPI) low at reset."
