File: hardware/console-s3/console-s3/console-s3.kicad_sch (KiCad schematic)
At the start: 43 parts, among them J1 USB-C, J2 PANEL, Q1 S8050, Q2 AO3401A, SW1 D0, SW2 D1, SW3 D2, SW4 BOOT, SW5 RESET, U1 ESP32-S3-WROOM-1-N8R2, U2 ATECC608C, U3 ME6211C33, U4 USBLC6-2SC6

Commit message: console-s3: U1's schematic MPN is the N8R2; the order plan's via count
- The schematic's U1 still named the N4R2 (C2913203, 4 MB) in its MPN and
  Description; its value, the board and the generator name the N8R2. The two
  lines now match what the generator writes. ERC 0, DRC 0, parity 0;
  tools/keypcb jlc passes.
- The order plan said 74 vias; the re-route left 72.

Co-Authored-By: Claude Opus 5.5 <noreply@anthropic.com>
Claude-Session: https://claude.ai/code/session_014mGuGD4x9Si2dmdRKbhRec
Parts:
- U1: MPN ESP32-S3-WROOM-1-N4R2 -> ESP32-S3-WROOM-1-N8R2
Changed lines of the file:
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@@
 (property "Footprint" "pqs3:ESP32-S3-WROOM-1" (at 147.32 85.09 0) (effects (font (size 1.27 1.27)) (hide yes)))
 (property "Datasheet" "https://www.espressif.com/sites/default/files/documentation/esp32-s3-wroom-1_wroom-1u_datasheet_en.pdf" (at 147.32 85.09 0) (effects (font (size 1.27 1.27)) (hide yes)))
-(property "MPN" "ESP32-S3-WROOM-1-N4R2" (at 147.32 85.09 0) (effects (font (size 1.27 1.27)) (hide yes)))
-(property "Description" "ESP32-S3 module, 4 MB flash, 2 MB quad PSRAM, on the back; JLCPCB C2913203 is Standard-only: hand-soldered" (at 147.32 85.09 0) (effects (font (size 1.27 1.27)) (hide yes)))
+(property "MPN" "ESP32-S3-WROOM-1-N8R2" (at 147.32 85.09 0) (effects (font (size 1.27 1.27)) (hide yes)))
+(property "Description" "ESP32-S3 module, 8 MB flash, 2 MB quad PSRAM, on the back; JLCPCB C2913204 is Standard-only: hand-soldered" (at 147.32 85.09 0) (effects (font (size 1.27 1.27)) (hide yes)))
 (pin "1") (pin "2") (pin "3") (pin "4") (pin "5") (pin "6") (pin "7") (pin "8") (pin "9") (pin "10") (pin "11") (pin "12") (pin "13") (pin "14") (pin "15") (pin "16") (pin "17") (pin "18") (pin "19") (pin "20") (pin "21") (pin "22") (pin "23") (pin "24") (pin "25") (pin "26") (pin "27") (pin "28") (pin "29") (pin "30") (pin "31") (pin "32") (pin "33") (pin "34") (pin "35") (pin "36") (pin "37") (pin "38") (pin "39") (pin "40") (pin "41")
 (instances (project "console-s3" (path "/be27dd74-f3aa-4475-8fca-ee9b571b0799" (reference "U1") (unit 1)))))
