File: hardware/picoquorum-key/hardware/picoquorum-key/picoquorum-key.kicad_pcb (KiCad board)
At the start: 2 copper layers, 44 x 53 mm, 52 parts, among them J1 USB-C, J2 ST7789 1.14in panel, Q1 AO3401A, Q2 MMBT3904, SW1 D0 Reject, SW2 D1 Next, SW3 D2 Sign, SW6 BOOT, SW7 RESET, U1 ESP32-S3-WROOM-1-N8R2, U2 ATECC608C-MAHDA, U3 AMS1117-3.3, U4 USBLC6-2SC6

Commit message: picoquorum-key rev B: an optional key port for a key-c
Adds a straddle USB-C plug (C3151751) at the board's top-left corner, on a
0.8 mm board widened 6 mm to 50 x 53. The key-c gets an I2C bus of its own
(GPIO38/39) and power through an AP22653 switch whose EN is pulled down, so
the key is off at reset and under any image that doesn't know the port. The
port also has CC on GPIO1 (R17 47k on every board), ESD on every plug line,
and a TVS on VKEY.

Departures from the plan:
- No LED or FAULT pins. Rev A's routing closes in module pins 21 and 24.
  D4 and a key-c P3's LED run off VKEY, and U5's FAULT is left open.
- The ESP32 module footprint's 48 mm keep-out is removed. The antenna rule
  area is now the module's antenna end plus 0.5 mm.

Routing:
- Rev A's routing is copied, moved 6 mm and locked (seed_route.py), and
  Freerouting routes only the port's connections.
- finish_route.py routes the few connections it left open.
- One GND via by U6 was placed by hand.

Fit groups: bom.csv/cpl.csv for base boards, bom-port.csv/cpl-port.csv
with the port's parts. The Gerbers are the same for both.

Checks:
- ERC 0; DRC 0 violations, 0 unconnected, 0 parity.
- tools/test.sh: 161 tests, 11 skipped (test_3d: no FreeCAD here).
- Visual goldens re-approved (KiCad 10.0.7).

The console image (firmware/board.py) is unchanged: only this board's
profile constants, PINS.md and smoke test know the port.

Co-Authored-By: Claude Opus 5.5 <noreply@anthropic.com>
Claude-Session: https://claude.ai/code/session_01H2mKC2z3aivAd8yF8tbg6X
Parts:
- added C10: 10u, Capacitor_SMD:C_0805_2012Metric, F.Cu at (104.0, 100.8)
- added C9: 100n, Capacitor_SMD:C_0603_1608Metric, F.Cu at (104.0, 95.4)
- added D3: ESD5Z5V0, Diode_SMD:D_SOD-523, F.Cu at (102.2, 65.6)
- added D4: green, LED_SMD:LED_0603_1608Metric, F.Cu at (102.2, 71.0)
- added J3: USB-C plug, straddle, console:USB_C_Plug_ShouHan_24P-GTJB_Straddle, F.Cu at (108.0, 60.0)
- added R15: 100k, Resistor_SMD:R_0603_1608Metric, F.Cu at (107.6, 97.0)
- added R17: 47k, Resistor_SMD:R_0603_1608Metric, F.Cu at (125.4, 63.4)
- added R18: 1k, Resistor_SMD:R_0603_1608Metric, F.Cu at (123.6, 63.4)
- added R19: 2.2k, Resistor_SMD:R_0603_1608Metric, F.Cu at (106.4, 103.4)
- added R20: 2.2k, Resistor_SMD:R_0603_1608Metric, F.Cu at (106.4, 105.2)
- added R21: 100, Resistor_SMD:R_0603_1608Metric, F.Cu at (102.2, 67.4)
- added R22: 1k, Resistor_SMD:R_0603_1608Metric, F.Cu at (102.2, 69.2)
- added TP13: KEY2_SDA, TestPoint:TestPoint_Pad_1.5x1.5mm, B.Cu at (108.4, 103.0)
- added TP14: KEY2_SCL, TestPoint:TestPoint_Pad_1.5x1.5mm, B.Cu at (115.0, 103.0)
- added U5: AP22653W6-7, Package_TO_SOT_SMD:SOT-23-6, F.Cu at (104.0, 98.0)
- added U6: USBLC6-2SC6, Package_TO_SOT_SMD:SOT-23-6, F.Cu at (116.6, 64.6)
- added U7: USBLC6-2SC6, Package_TO_SOT_SMD:SOT-23-6, F.Cu at (120.8, 64.6)
- TP10: value IO2 -> KEY_EN
- TP9: value IO1 -> KEY_CC
- moved C1 6.00 mm to (111.0, 106.0)
- moved C2 6.00 mm to (119.3, 104.2)
- moved C3 6.00 mm to (146.8, 69.6)
- moved C4 6.00 mm to (147.0, 72.8)
- moved C5 6.00 mm to (148.8, 69.6)
- moved C6 6.00 mm to (123.8, 80.2)
- moved C7 6.00 mm to (142.6, 89.2)
- moved C8 6.00 mm to (113.2, 106.0)
- moved D1 6.00 mm to (131.5, 89.0)
- moved H2 6.00 mm to (147.0, 89.5)
- moved H4 6.00 mm to (147.0, 110.0)
- moved J1 6.00 mm to (128.0, 109.3)
- moved J2 6.00 mm to (126.5, 77.3)
- moved Q1 6.00 mm to (121.0, 90.0)
- moved Q2 6.00 mm to (121.0, 94.0)
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Connections:
- net IO1 renamed KEY_CC
- net IO2 renamed KEY_EN
- U1 pad 31: unconnected-(U1-IO38-Pad31) -> KEY2_SDA
- U1 pad 32: unconnected-(U1-IO39-Pad32) -> KEY2_SCL
Routing:
- net KEY2_SDA: track 0.00 -> 131.8 mm, vias 0 -> 7
- net KEY2_SCL: track 0.00 -> 100.4 mm, vias 0 -> 9
- net GND: track 274.5 -> 368.0 mm, vias 62 -> 65
- net VKEY: track 0.00 -> 78.3 mm, vias 0 -> 6
- net +3V3: track 126.5 -> 175.7 mm, vias 7 -> 12
- net KEY_EN: track 42.1 -> 85.0 mm, vias 2 -> 4
- net KEY_SBU: track 0.00 -> 34.9 mm, vias 0 -> 5
- net KEY_CC: track 59.0 -> 86.2 mm, vias 4 -> 3
- net KEY_CC_PLUG: track 0.00 -> 24.5 mm, vias 0 -> 2
- net KEY_LED_A: track 0.00 -> 1.82 mm
- net USB_DN: track 15.9 -> 17.5 mm
Other:
- board size 44 x 53 mm -> 50 x 53 mm
- board text added: "KCC"
- board text added: "KEN"
- board text added: "KEY PORT"
- board text added: "KEY, REV B"
- board text added: "KSCL"
- board text added: "KSDA"
- board text removed: "IO1"
- board text removed: "IO2"
- board text removed: "KEY, REV A"
- board text removed: "ONE KEY"

Commit message: picoquorum-key rev B: D4 is D1's red LED (C2286)
The plan's green LED (C72043) is out of stock at JLCPCB. D4 is now the
red KT-0603R that D1 already uses: a basic part already on every order,
so no extra BOM line. At 3.3 V through R22 (1k) it gets about 1.4 mA, as
D1 does; the green InGaN part would have got under 1 mA.

Checks: ERC 0, DRC 0, tools/test.sh OK (11 skipped: no FreeCAD).

Co-Authored-By: Claude Opus 5.5 <noreply@anthropic.com>
Claude-Session: https://claude.ai/code/session_01H2mKC2z3aivAd8yF8tbg6X
Parts:
- D4: value green -> red
Changed lines of the file:
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@@
 			)
 		)
-		(property "Value" "green"
+		(property "Value" "red"
 			(at 0 1.43 0)
 			(layer "F.Fab")
@@
 			)
 		)
-		(property "LCSC" "C72043"
+		(property "LCSC" "C2286"
 			(at 0 0 0)
 			(layer "F.SilkS")
@@
 			)
 		)
-		(property "MPN" "19-217/GHC-YR1S2/3T"
+		(property "MPN" "KT-0603R"
 			(at 0 0 0)
 			(layer "F.SilkS")

Commit message: picoquorum-key rev B: D4 is a green KT-0603G (C12624)
Replaces the red C2286 stand-in. The plan's green C72043 is out of stock.
C12624's JLCPCB tier and stock weren't checked from here. At 3.3 V
through R22 (1k) a green LED gets under 1 mA; BRINGUP.md says to drop
R22 to 470 ohm if it is too dim.

Checks: ERC 0, DRC 0, tools/test.sh OK (11 skipped: no FreeCAD).

Co-Authored-By: Claude Opus 5.5 <noreply@anthropic.com>
Claude-Session: https://claude.ai/code/session_01H2mKC2z3aivAd8yF8tbg6X
Parts:
- D4: value red -> green
Changed lines of the file:
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@@
 			)
 		)
-		(property "Value" "red"
+		(property "Value" "green"
 			(at 0 1.43 0)
 			(layer "F.Fab")
@@
 			)
 		)
-		(property "LCSC" "C2286"
+		(property "LCSC" "C12624"
 			(at 0 0 0)
 			(layer "F.SilkS")
@@
 			)
 		)
-		(property "MPN" "KT-0603R"
+		(property "MPN" "KT-0603G"
 			(at 0 0 0)
 			(layer "F.SilkS")

Commit message: picoquorum-key rev B: R22 470 ohm (C23179) for D4
The green KT-0603G drops about 2.7 V or more, so through 1k from VKEY it
got under 1 mA. 470 ohm gives about 1 mA. R22 is no longer on R18's 1k line,
so bom-port.csv has one line more.

Checks: ERC 0, DRC 0, tools/test.sh OK (11 skipped: no FreeCAD).

Co-Authored-By: Claude Opus 5.5 <noreply@anthropic.com>
Claude-Session: https://claude.ai/code/session_01H2mKC2z3aivAd8yF8tbg6X
Parts:
- R22: value 1k -> 470
Changed lines of the file:
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@@
 			)
 		)
-		(property "Value" "1k"
+		(property "Value" "470"
 			(at 0 1.43 0)
 			(layer "F.Fab")
@@
 			)
 		)
-		(property "LCSC" "C21190"
+		(property "LCSC" "C23179"
 			(at 0 0 0)
 			(layer "F.SilkS")
@@
 			)
 		)
-		(property "MPN" "1k"
+		(property "MPN" "470"
 			(at 0 0 0)
 			(layer "F.SilkS")

Commit message: picoquorum-key rev B: 5 V on the key port's VBUS no longer reaches 3V3 through SBU
U7's second channel was on SBU, which R21 (100 ohm) feeds from VKEY.
5 V put on the plug's VBUS then went R21 -> U7's diode -> 3V3, around
U5's reverse blocking: about 11 mA with the board on, enough to
half-power it when off. U7 now covers CC only; SBU meets only R21, so
D3 clamps it through 100 ohm. Its spur (3 vias, 13 segments) is gone
from the board; nothing else moved.

What is left is R19/R20 (2.2k) into U6's diodes and GPIO38/39's
clamps, about 0.5 mA a line. test_key_port holds the board to that,
and fails on the old circuit. BRINGUP.md gets a bench-supply check.

DESIGN.md's regulator note said the AMS1117 "wants >= 10 uF for
stability". Its datasheet asks for 22 uF of solid tantalum for all
conditions, allows smaller without an ADJ capacitor, and says nothing
about ceramics, which is all this board has. The note now says so,
with the heat sum, and BRINGUP.md scopes 3V3. The parts are unchanged.

ERC 0, DRC 0 with schematic parity. tools/test.sh: 162 tests, one
failure, test_3d's J3 without a model, as before. Fab files and the
approved pictures remade with KiCad 10.0.6 (they were 10.0.7's).

Co-Authored-By: Claude Opus 5.5 <noreply@anthropic.com>
Claude-Session: https://claude.ai/code/session_015Mrfds5ggPmPXMnhiEk5Pk
Connections:
- U7 pad 3: KEY_SBU -> unconnected-(U7-I/O2-Pad3)
- U7 pad 4: KEY_SBU -> unconnected-(U7-I/O2-Pad4)
Routing:
- net KEY_SBU: track 34.9 -> 19.2 mm, vias 5 -> 2
Changed lines of the file:
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@@
 			)
 		)
-		(property "Description" "ESD on CC and the LED line (SBU), at the plug; its rail on 3V3"
+		(property "Description" "ESD on CC, at the plug; its rail on 3V3. Not on SBU: R21 would feed 5 V on VBUS into 3V3"
 			(at 0 0 0)
 			(layer "F.Fab")
@@
 			(layers "F.Cu" "F.Mask" "F.Paste")
 			(roundrect_rratio 0.25)
-			(net "KEY_SBU")
+			(net "unconnected-(U7-I{slash}O2-Pad3)")
 		)
 		(pad "4" smd roundrect
@@
 			(layers "F.Cu" "F.Mask" "F.Paste")
 			(roundrect_rratio 0.25)
-			(net "KEY_SBU")
+			(net "unconnected-(U7-I{slash}O2-Pad4)")
 		)
 		(pad "5" smd roundrect
@@
 	)
 	(segment
-		(start 121.7608 65.7267)
-		(end 121.9375 65.55)
-		(width 0.25)
-		(layer "F.Cu")
-		(net "KEY_SBU")
-	)
-	(segment
 		(start 109.7742 65.129)
 		(end 110.0059 65.3607)
@@
 	)
 	(segment
-		(start 119.6625 65.55)
-		(end 118.8038 66.4087)
-		(width 0.25)
-		(layer "F.Cu")
-		(net "KEY_SBU")
-	)
-	(segment
 		(start 108.75 61.95)
 		(end 108.75 64.0118)
@@
 	)
 	(segment
-		(start 118.3507 66.4087)
-		(end 116.7029 66.4087)
-		(width 0.25)
-		(layer "F.Cu")
-		(net "KEY_SBU")
-	)
-	(segment
 		(start 103.866 67.4)
 		(end 104.054 67.588)
@@
 	)
 	(segment
-		(start 118.8038 66.4087)
-		(end 118.3507 66.4087)
-		(width 0.25)
-		(layer "F.Cu")
-		(net "KEY_SBU")
-	)
-	(segment
-		(start 118.3507 66.4087)
-		(end 118.3507 66.9517)
-		(width 0.25)
-		(layer "F.Cu")
-		(net "KEY_SBU")
-	)
-	(segment
-		(start 121.7608 66.6707)
-		(end 121.7608 65.7267)
-		(width 0.25)
-		(layer "F.Cu")
-		(net "KEY_SBU")
-	)
-	(segment
 		(start 103.025 67.4)
 		(end 103.866 67.4)
@@
 	)
 	(via
-		(at 121.7608 66.6707)
-		(size 0.6)
-		(drill 0.3)
-		(layers "F.Cu" "B.Cu")
-		(net "KEY_SBU")
-	)
-	(via
-		(at 116.7029 66.4087)
-		(size 0.6)
-		(drill 0.3)
-		(layers "F.Cu" "B.Cu")
-		(net "KEY_SBU")
-	)
-	(via
 		(at 104.054 67.588)
 		(size 0.6)
@@
 		(net "KEY_SBU")
 	)
-	(via
-		(at 118.3507 66.9517)
-		(size 0.6)
-		(drill 0.3)
-		(layers "F.Cu" "B.Cu")
-		(net "KEY_SBU")
-	)
-	(segment
-		(start 110.0059 67.588)
-		(end 115.5236 67.588)
-		(width 0.25)
-		(layer "B.Cu")
-		(net "KEY_SBU")
-	)
 	(segment
 		(start 106.4611 67.588)
@@
 	)
 	(segment
-		(start 115.5236 67.588)
-		(end 116.7029 66.4087)
-		(width 0.25)
-		(layer "B.Cu")
-		(net "KEY_SBU")
-	)
-	(segment
-		(start 118.3507 66.9517)
-		(end 121.4798 66.9517)
-		(width 0.25)
-		(layer "B.Cu")
-		(net "KEY_SBU")
-	)
-	(segment
 		(start 107.25 65.8516)
 		(end 106.4611 66.6405)
@@
 		(width 0.25)
 		(layer "B.Cu")
-		(net "KEY_SBU")
-	)
-	(segment
-		(start 121.4798 66.9517)
-		(end 121.7608 66.6707)
-		(width 0.25)
-		(layer "B.Cu")
