File: hardware/picoquorum-key/hardware/picoquorum-key/picoquorum-key.kicad_sch (KiCad schematic)
At the start: 69 parts, among them J1 USB-C, J2 ST7789 1.14in panel, J3 USB-C plug, straddle, Q1 AO3401A, Q2 MMBT3904, SW1 D0 Reject, SW2 D1 Next, SW3 D2 Sign, SW6 BOOT, SW7 RESET, U1 ESP32-S3-WROOM-1-N8R2, U2 ATECC608C-MAHDA, U3 AMS1117-3.3, U4 USBLC6-2SC6, U5 AP22653W6-7, U6 USBLC6-2SC6, U7 USBLC6-2SC6

Commit message: picoquorum-key rev B: D5, a Schottky between U5 and the plug
U5 (AP22653) blocks reverse current only while off; on, it limits it
to 0.32 A, which would push 3V3 past the S3's 3.6 V if 5 V reached the
plug's VBUS. D5 (1N5819WS, C191023, basic) now sits between U5's output
(new net VKEY_SW) and VKEY: 5 V on the plug stops there, U5 on or off.
About 0.2 V of drop at the key's current, so the key sees ~3.1 V.

- R19/R20 move to VKEY_SW: a key that is off still isn't fed through
  its bus, and 5 V on the plug no longer reaches GPIO38/39's clamps.
- R23 (10k) drains VKEY, which U5's discharge can't reach through D5.
- Board: D5 and R23 in VKEY's run up the left strip (4, 19.5) and
  (2.2, 19.5); the track was cut for D5, four ground stitching vias
  made room, R23's ground pad has its own via. Nothing else moved.
- PINS.md drops the GPIO38/39 check before enabling: it is not needed.
- test_key_port: nothing on VKEY leads to 3V3 or VKEY_SW but D5.
  test_spice and the twin follow the pull-ups to VKEY_SW.
- DESIGN.md: why not U5 alone, the AP22653A or the TPS22917 (its
  blocking needs 0.5 A of reverse current first). Open: the ATECC608C's
  pin limit, with the bus at 3.3 V and the key at ~3.1 V.

ERC 0, DRC 0 with schematic parity. Port BOM/CPL gain D5 and R23; the
base BOM is unchanged. tools/test.sh: 162 tests, one failure, test_3d's
J3 without a model, as before. Approved pictures remade (KiCad 10.0.6).

Co-Authored-By: Claude Opus 5.5 <noreply@anthropic.com>
Claude-Session: https://claude.ai/code/session_015Mrfds5ggPmPXMnhiEk5Pk
Parts:
- added D5: 1N5819WS, Diode_SMD:D_SOD-323, symbol Device:D_Schottky
- added R23: 10k, Resistor_SMD:R_0603_1608Metric, symbol Device:R
Connections:
- net GND: now also R23.2
- net VKEY: now also D5.1 (K), R23.1; no longer C10.1, R19.1, R20.1, U5.6 (OUT)
- new net VKEY_SW: C10.1, D5.2 (A), R19.1, R20.1, U5.6 (OUT)
Other:
- note added: "7 THE KEY PORT (rev B): a key-c on its own bus, I2C(1) Fit 'port' only, but R17 (every board). Power off at reset: R15 holds U5's EN low. D5 from U5's output to VKEY: 5 V on the plug stops there, U5 on or off. R23 drains VKEY. SDA on D+ (A6), SCL on D- (A7), VKEY on VBUS, one CC line (A5), SBU (A8+B8) from VKEY. ESD rails on 3V3, never VKEY; none on SBU (R21, D3 cover it). J3 hand-fitted; 0.8 mm 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"
- note removed: "7 THE KEY PORT (rev B): a key-c on its own bus, I2C(1) Fit 'port' only, but R17 (every board). Power off at reset: R15 holds U5's EN low. SDA on D+ (A6), SCL on D- (A7), VKEY on VBUS, one CC line (A5), SBU (A8+B8) from VKEY. ESD rails on 3V3, never VKEY; none on SBU (R21, D3 cover it). J3 hand-fitted; 0.8 mm board."
